File: multi-pcb-cpu.sch (EAGLE design)
At the start: 9 parts

Commit message: Made schematic more compact/clean
Parts:
- removed DISPLAY: 2.54B-ZR, con-jst-custom:2.54B-ZR
- removed JP_I2C_1, JP_I2C_2, JP_UART0: (no value), pinhead:PINHD-1X4
- removed JP_SPI_1: (no value), pinhead:PINHD-2X3
- added JP_CRUISE_CONTROL, JP_UART_GPS: 6B-ZR, con-jst-custom:6B-ZR
- added JP_I2C0_9AXIS_SENSOR, JP_I2C1_DISPLAY, JP_POWER: 2.54B-ZR, con-jst-custom:2.54B-ZR
- added JP_I2C0_EXTRA, JP_UART_EXTRA: (no value), pinhead:PINHD-1X4
- added JP_SPI_EXTRA: (no value), pinhead:PINHD-2X3
- added JP_SPI_OTHER: 8B-ZR, con-jst-custom:8B-ZR
- added JP_SWITCHES: 2.55B-ZR, con-jst-custom:2.55B-ZR
Connections:
- net +3V3: now also JP_I2C0_9AXIS_SENSOR-4.1, JP_I2C1_DISPLAY-4.1, JP_POWER-3.1, JP_SWITCHES-5.1, JP_UART_GPS-5.1; no longer DISPLAY-4.1
- net +5V: now also JP_CRUISE_CONTROL-6.1, JP_I2C0_EXTRA.4, JP_POWER-4.1, JP_SPI_EXTRA.2, JP_SPI_OTHER-8.1, JP_UART_EXTRA.4, JP_UART_GPS-6.1; no longer JP_I2C_1.4, JP_I2C_2.4, JP_SPI_1.2, JP_UART0.4
- net APP_ENABLE: now also JP_CRUISE_CONTROL-5.1
- net APP_PWM_OUT_0: now also JP_CRUISE_CONTROL-4.1
- net APP_PWM_OUT_1: now also JP_CRUISE_CONTROL-3.1
- net BTN_0: now also JP_SWITCHES-4.1
- net BTN_1: now also JP_SWITCHES-3.1
- net CAN_CS: now also JP_SPI_OTHER-3.1
- net CAN_INT: now also JP_SPI_OTHER-2.1
- net CLAXON_ENABLE: now also JP_SWITCHES-1.1
- net ENGINE_CUTOFF_DISABLE: now also JP_SWITCHES-2.1
- net GND: now also JP_I2C0_9AXIS_SENSOR-1.1, JP_I2C0_EXTRA.1, JP_I2C1_DISPLAY-1.1, JP_POWER-1.1, JP_SPI_EXTRA.6, JP_SPI_OTHER-1.1, JP_UART_EXTRA.1, JP_UART_GPS-1.1; no longer DISPLAY-1.1, JP_I2C_1.1, JP_I2C_2.1, JP_SPI_1.6, JP_UART0.1
- net I2C0_SCL: now also JP_I2C0_9AXIS_SENSOR-3.1, JP_I2C0_EXTRA.3; no longer JP_I2C_1.3, JP_I2C_2.3
- net I2C0_SDA: now also JP_I2C0_9AXIS_SENSOR-2.1, JP_I2C0_EXTRA.2; no longer JP_I2C_1.2, JP_I2C_2.2
- net I2C1_SCL: now also JP_I2C1_DISPLAY-3.1; no longer DISPLAY-3.1
- net I2C1_SDA: now also JP_I2C1_DISPLAY-2.1; no longer DISPLAY-2.1
- net MCU_RESET: now also JP_UART_GPS-2.1
- net PWR_ENABLE: now also JP_POWER-2.1
- net SD_CS: now also JP_SPI_OTHER-4.1
- net SENS_APP_0_IN: now also JP_CRUISE_CONTROL-2.1
- net SENS_APP_1_IN: now also JP_CRUISE_CONTROL-1.1
- net SPI_CS_1: now also JP_SPI_EXTRA.5; no longer JP_SPI_1.5
- net SPI_MISO_5V: now also JP_SPI_EXTRA.1, JP_SPI_OTHER-7.1; no longer JP_SPI_1.1
- net SPI_MOSI: now also JP_SPI_EXTRA.4, JP_SPI_OTHER-6.1; no longer JP_SPI_1.4
- net SPI_SCK: now also JP_SPI_EXTRA.3, JP_SPI_OTHER-5.1; no longer JP_SPI_1.3
- net UART0_RX: now also JP_UART_EXTRA.3; no longer JP_UART0.3
- net UART0_TX: now also JP_UART_EXTRA.2; no longer JP_UART0.2
- net UART2_RX: now also JP_UART_GPS-3.1
- net UART2_TX: now also JP_UART_GPS-4.1
Other:
- moved on the sheet: R24, R25, RESET, U$1

Commit message: updated some PCB's
Parts:
- R24: value 5k -> 0
- R25: value 10k -> 1.8k
Connections:
- net CAN_CS: now also JP_SPI_OTHER-4.1; no longer JP_SPI_OTHER-3.1
- net CAN_INT: now also JP_SPI_OTHER-3.1; no longer JP_SPI_OTHER-2.1
- net MCU_RESET: now also JP_UART_GPS-4.1; no longer JP_UART_GPS-2.1
- net SD_CS: now also JP_SPI_OTHER-2.1; no longer JP_SPI_OTHER-4.1
- net SPI_MISO_5V: now also JP_SPI_OTHER-5.1; no longer JP_SPI_OTHER-7.1
- net SPI_SCK: now also JP_SPI_OTHER-7.1; no longer JP_SPI_OTHER-5.1
- net UART2_TX: now also JP_UART_GPS-2.1; no longer JP_UART_GPS-4.1
Changed lines of the file:
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@@
 <part name="+3V4" library="supply1" library_urn="urn:adsk.eagle:library:371" deviceset="+3V3" device=""/>
 <part name="GND22" library="supply1" library_urn="urn:adsk.eagle:library:371" deviceset="GND" device=""/>
-<part name="R24" library="rcl" library_urn="urn:adsk.eagle:library:334" deviceset="R-EU_" device="0207/7" package3d_urn="urn:adsk.eagle:package:23493/2" value="5k"/>
-<part name="R25" library="rcl" library_urn="urn:adsk.eagle:library:334" deviceset="R-EU_" device="0207/7" package3d_urn="urn:adsk.eagle:package:23493/2" value="10k"/>
+<part name="R24" library="rcl" library_urn="urn:adsk.eagle:library:334" deviceset="R-EU_" device="0207/7" package3d_urn="urn:adsk.eagle:package:23493/2" value="0"/>
+<part name="R25" library="rcl" library_urn="urn:adsk.eagle:library:334" deviceset="R-EU_" device="0207/7" package3d_urn="urn:adsk.eagle:package:23493/2" value="1.8k"/>
 <part name="GND3" library="supply1" library_urn="urn:adsk.eagle:library:371" deviceset="GND" device=""/>
 <part name="P+1" library="supply1" library_urn="urn:adsk.eagle:library:371" deviceset="+5V" device=""/>
@@
 <net name="CAN_CS" class="0">
 <segment>
+<label x="-177.8" y="-58.42" size="1.778" layer="95" xref="yes"/>
+<pinref part="JP_SPI_OTHER" gate="-4" pin="1"/>
+<wire x1="-182.88" y1="-58.42" x2="-177.8" y2="-58.42" width="0.1524" layer="91"/>
+</segment>
+<segment>
 <pinref part="U$1" gate="G$1" pin="IO2"/>
 <wire x1="-38.1" y1="17.78" x2="-35.56" y2="17.78" width="0.1524" layer="91"/>
 <label x="-35.56" y="17.78" size="1.778" layer="95" xref="yes"/>
-</segment>
-<segment>
-<label x="-177.8" y="-60.96" size="1.778" layer="95" xref="yes"/>
-<wire x1="-177.8" y1="-60.96" x2="-175.26" y2="-58.42" width="0.1524" layer="91"/>
-<pinref part="JP_SPI_OTHER" gate="-3" pin="1"/>
-<wire x1="-182.88" y1="-60.96" x2="-177.8" y2="-60.96" width="0.1524" layer="91"/>
 </segment>
 </net>
@@
 <segment>
 <label x="-177.8" y="-53.34" size="1.778" layer="95" xref="yes"/>
-<wire x1="-177.8" y1="-53.34" x2="-175.26" y2="-50.8" width="0.1524" layer="91"/>
 <pinref part="JP_SPI_OTHER" gate="-6" pin="1"/>
 <wire x1="-182.88" y1="-53.34" x2="-177.8" y2="-53.34" width="0.1524" layer="91"/>
@@
 </segment>
 <segment>
-<label x="-177.8" y="-55.88" size="1.778" layer="95" xref="yes"/>
-<wire x1="-177.8" y1="-55.88" x2="-175.26" y2="-53.34" width="0.1524" layer="91"/>
-<pinref part="JP_SPI_OTHER" gate="-5" pin="1"/>
-<wire x1="-182.88" y1="-55.88" x2="-177.8" y2="-55.88" width="0.1524" layer="91"/>
+<label x="-177.8" y="-50.8" size="1.778" layer="95" xref="yes"/>
+<pinref part="JP_SPI_OTHER" gate="-7" pin="1"/>
+<wire x1="-182.88" y1="-50.8" x2="-177.8" y2="-50.8" width="0.1524" layer="91"/>
 </segment>
 </net>
 <net name="CAN_INT" class="0">
+<segment>
+<label x="-177.8" y="-60.96" size="1.778" layer="95" xref="yes"/>
+<pinref part="JP_SPI_OTHER" gate="-3" pin="1"/>
+<wire x1="-182.88" y1="-60.96" x2="-177.8" y2="-60.96" width="0.1524" layer="91"/>
+</segment>
 <segment>
 <pinref part="U$1" gate="G$1" pin="IO4"/>
@@
 <label x="-35.56" y="20.32" size="1.778" layer="95" xref="yes"/>
 </segment>
-<segment>
-<label x="-177.8" y="-63.5" size="1.778" layer="95" xref="yes"/>
-<wire x1="-177.8" y1="-63.5" x2="-175.26" y2="-60.96" width="0.1524" layer="91"/>
-<pinref part="JP_SPI_OTHER" gate="-2" pin="1"/>
-<wire x1="-182.88" y1="-63.5" x2="-177.8" y2="-63.5" width="0.1524" layer="91"/>
-</segment>
 </net>
 <net name="I2C0_SDA" class="0">
@@
 </segment>
 <segment>
-<label x="-177.8" y="-20.32" size="1.778" layer="95" xref="yes"/>
-<pinref part="JP_UART_GPS" gate="-4" pin="1"/>
-<wire x1="-182.88" y1="-20.32" x2="-177.8" y2="-20.32" width="0.1524" layer="91"/>
+<label x="-177.8" y="-25.4" size="1.778" layer="95" xref="yes"/>
+<pinref part="JP_UART_GPS" gate="-2" pin="1"/>
+<wire x1="-177.8" y1="-25.4" x2="-182.88" y2="-25.4" width="0.1524" layer="91"/>
 </segment>
 </net>
@@
 </segment>
 <segment>
-<label x="-177.8" y="-58.42" size="1.778" layer="95" xref="yes"/>
-<wire x1="-177.8" y1="-58.42" x2="-175.26" y2="-55.88" width="0.1524" layer="91"/>
-<pinref part="JP_SPI_OTHER" gate="-4" pin="1"/>
-<wire x1="-182.88" y1="-58.42" x2="-177.8" y2="-58.42" width="0.1524" layer="91"/>
+<label x="-177.8" y="-63.5" size="1.778" layer="95" xref="yes"/>
+<pinref part="JP_SPI_OTHER" gate="-2" pin="1"/>
+<wire x1="-182.88" y1="-63.5" x2="-177.8" y2="-63.5" width="0.1524" layer="91"/>
 </segment>
 </net>
@@
 </segment>
 <segment>
-<label x="-177.8" y="-25.4" size="1.778" layer="95" xref="yes"/>
-<pinref part="JP_UART_GPS" gate="-2" pin="1"/>
-<wire x1="-177.8" y1="-25.4" x2="-182.88" y2="-25.4" width="0.1524" layer="91"/>
+<label x="-177.8" y="-20.32" size="1.778" layer="95" xref="yes"/>
+<pinref part="JP_UART_GPS" gate="-4" pin="1"/>
+<wire x1="-182.88" y1="-20.32" x2="-177.8" y2="-20.32" width="0.1524" layer="91"/>
 </segment>
 </net>
@@
 </segment>
 <segment>
-<label x="-177.8" y="-50.8" size="1.778" layer="95" xref="yes"/>
-<wire x1="-177.8" y1="-50.8" x2="-175.26" y2="-48.26" width="0.1524" layer="91"/>
-<pinref part="JP_SPI_OTHER" gate="-7" pin="1"/>
-<wire x1="-182.88" y1="-50.8" x2="-177.8" y2="-50.8" width="0.1524" layer="91"/>
-</segment>
-</net>
+<label x="-177.8" y="-55.88" size="1.778" layer="95" xref="yes"/>
+<pinref part="JP_SPI_OTHER" gate="-5" pin="1"/>
+<wire x1="-182.88" y1="-55.88" x2="-177.8" y2="-55.88" width="0.1524" layer="91"/>
+</segment>
+</net>
