File: multi-pcb-cruisecontrol.brd (EAGLE design)
At the start: 77.1 x 28.6 mm, 28 parts, among them IC1 LM358N, K1 351, T1 BC618, X1 2.52B-ZR, X2 2.52B-ZR, X4 6B-ZR, X5 2.52B-ZR

Commit message: updated some PCB's
Parts:
- R10, R11, R8, R9: value 10k -> 220k
Changed lines of the file:
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@@
 <layer number="23" name="tOrigins" color="15" fill="1" visible="yes" active="yes"/>
 <layer number="24" name="bOrigins" color="15" fill="1" visible="yes" active="yes"/>
-<layer number="25" name="tNames" color="7" fill="1" visible="no" active="yes"/>
+<layer number="25" name="tNames" color="7" fill="1" visible="yes" active="yes"/>
 <layer number="26" name="bNames" color="7" fill="1" visible="yes" active="yes"/>
 <layer number="27" name="tValues" color="7" fill="1" visible="no" active="yes"/>
@@
 <attribute name="VALUE" x="19.05" y="17.5133" size="1.27" layer="27" ratio="10" rot="R180"/>
 </element>
-<element name="R10" library="rcl" library_urn="urn:adsk.eagle:library:334" package="0207/7" package3d_urn="urn:adsk.eagle:package:23493/2" value="10k" x="18.7325" y="2.54" smashed="yes">
+<element name="R10" library="rcl" library_urn="urn:adsk.eagle:library:334" package="0207/7" package3d_urn="urn:adsk.eagle:package:23493/2" value="220k" x="18.7325" y="2.54" smashed="yes">
 <attribute name="NAME" x="16.1925" y="3.937" size="1.27" layer="25" ratio="10"/>
 <attribute name="POPULARITY" value="46" x="56.8325" y="-72.39" size="1.778" layer="27" display="off"/>
@@
 <attribute name="VALUE" x="16.4465" y="1.9812" size="1.27" layer="27" ratio="10"/>
 </element>
-<element name="R11" library="rcl" library_urn="urn:adsk.eagle:library:334" package="0207/7" package3d_urn="urn:adsk.eagle:package:23493/2" value="10k" x="46.355" y="2.54" smashed="yes">
+<element name="R11" library="rcl" library_urn="urn:adsk.eagle:library:334" package="0207/7" package3d_urn="urn:adsk.eagle:package:23493/2" value="220k" x="46.355" y="2.54" smashed="yes">
 <attribute name="NAME" x="42.164" y="4.445" size="1.27" layer="25" ratio="10"/>
 <attribute name="POPULARITY" value="46" x="65.405" y="-67.31" size="1.778" layer="27" display="off"/>
@@
 <attribute name="VALUE" x="27.686" y="21.5138" size="1.27" layer="27" ratio="10" rot="R180"/>
 </element>
-<element name="R8" library="rcl" library_urn="urn:adsk.eagle:library:334" package="0207/7" package3d_urn="urn:adsk.eagle:package:23493/2" value="10k" x="29.845" y="5.08" smashed="yes">
+<element name="R8" library="rcl" library_urn="urn:adsk.eagle:library:334" package="0207/7" package3d_urn="urn:adsk.eagle:package:23493/2" value="220k" x="29.845" y="5.08" smashed="yes">
 <attribute name="NAME" x="27.305" y="6.477" size="1.27" layer="25" ratio="10"/>
 <attribute name="POPULARITY" value="46" x="57.785" y="-69.85" size="1.778" layer="27" display="off"/>
@@
 <attribute name="VALUE" x="27.559" y="4.5212" size="1.27" layer="27" ratio="10"/>
 </element>
-<element name="R9" library="rcl" library_urn="urn:adsk.eagle:library:334" package="0207/7" package3d_urn="urn:adsk.eagle:package:23493/2" value="10k" x="46.355" y="5.08" smashed="yes">
+<element name="R9" library="rcl" library_urn="urn:adsk.eagle:library:334" package="0207/7" package3d_urn="urn:adsk.eagle:package:23493/2" value="220k" x="46.355" y="5.08" smashed="yes">
 <attribute name="NAME" x="42.164" y="6.985" size="1.27" layer="25" ratio="10"/>
 <attribute name="POPULARITY" value="46" x="118.745" y="-58.42" size="1.778" layer="27" display="off"/>
